Commit message: work almost good with imu

File: src/xunjian_nav/urdf/test_model.urdf (robot description, URDF)
Before this commit: robot test_model, 2 links, 1 joints
Links:
- removed link laser_link
- added link laser; visual cylinder length=0.04 radius=0.03
- added link point; visual cylinder length=0.04 radius=0.03
Joints:
- added joint base_to_point: type fixed, parent base_link, child point, origin xyz=0 0 0
- joint base_to_laser: child laser_link -> laser
